File: 32U4Castel.sch (EAGLE design)
At the start: 19 parts, among them U1 ATMEGA32U4, Y1 16MHz

Commit message: Added pad, complete re-route
Fabrication was difficult because of non-ground vias where 32U4 wanted a pad. Added pad, rerouted everything. Improved silkscreen.
Parts:
- U1: device Testing:ATMEGA32U4OUTFAKES -> 32U4Castel:TESTING_ATMEGA32U4QFN
Other:
- moved on the sheet: U1
Changed lines of the file:
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@@
 <layer number="59" name="tCarbon" color="7" fill="1" visible="no" active="no"/>
 <layer number="60" name="bCarbon" color="7" fill="1" visible="no" active="no"/>
+<layer number="88" name="SimResults" color="9" fill="1" visible="yes" active="yes"/>
+<layer number="89" name="SimProbes" color="9" fill="1" visible="yes" active="yes"/>
 <layer number="90" name="Modules" color="5" fill="1" visible="yes" active="yes"/>
 <layer number="91" name="Nets" color="2" fill="1" visible="yes" active="yes"/>
@@
 <part name="GND7" library="SparkFun" deviceset="GND" device=""/>
 <part name="GND4" library="SparkFun" deviceset="GND" device=""/>
-<part name="U1" library="Testing" deviceset="ATMEGA32U4" device="OUTFAKES" value="ATMEGA32U4"/>
+<part name="U1" library="32U4Castel" deviceset="TESTING_ATMEGA32U4" device="QFN" value="ATMEGA32U4"/>
 <part name="Y1" library="SparkFun" deviceset="CRYSTAL" device="5X3" value="16MHz"/>
 <part name="C2" library="SparkFun" deviceset="CAP" device="0603-CAP" value="22pF"/>

Commit message: Updated 32U4Castel
Fixed mis-mapped SS pin and improved grounding.
Parts:
- added C10, C9: 1uF, SparkFun:CAP0603-CAP
- J1, J3: device SparkFun-Connectors:CONN_08NO_SILK_FEMALE_PTH -> SparkFun-Connectors:CONN_09NO_SILK
- U1: value ATMEGA32U4 -> ATMEGA32U4-MU; device 32U4Castel:TESTING_ATMEGA32U4QFN -> 32U4:ATMEGA32U4-MU
Connections:
- net N$1 renamed X2
- net N$2 renamed X1
- net N$38 renamed LED
- net N$4 renamed UCAP
- new net D14: J1.1, U1.PB0(SS)
- net D10: now also J1.5; no longer J3.4
- net D11: now also J1.4; no longer J3.3
- net D12: now also J1.3; no longer J3.2
- net D13: now also J1.2; no longer J3.1
- net D6: now also J1.9; no longer J3.8
- net D7: now also J1.8; no longer J3.7
- net D8: now also J1.7; no longer J3.6
- net D9: now also J1.6; no longer J3.5
- net GND: now also C10.1, C9.1, J3.4, U1.EPAD, U1.GND, U1.GND_2, U1.GND_3, U1.GND_4, U1.PE2; no longer J1.4, U1.GND@15, U1.GND@23, U1.GND@35, U1.GND@43, U1.PE2/!HWB
- net MISO: now also J3.7; no longer J1.5
- net MOSI: now also J3.6; no longer J1.7
- net RESET: now also J3.8; no longer J1.8
- net SCK: now also J3.5; no longer J1.6
- net VCC: now also C10.2, C9.2, J3.1, U1.AVCC, U1.AVCC_2, U1.VCC, U1.VCC_2; no longer J1.1, U1.AVCC@24, U1.AVCC@44, U1.VCC@14, U1.VCC@34
- net XD+: now also J3.3; no longer J1.3
- net XD-: now also J3.2; no longer J1.2
